File: VCO/VCO_pcb/VCO.kicad_pcb (KiCad board)
At the start: 2 copper layers, 30 x 108.5 mm, 67 parts, among them J1 Thonkiconn, J2 Thonkiconn, J3 Thonkiconn, J4 Thonkiconn, J5 Thonkiconn, Q1 BCM847BS,115, Q2 MMBFJ111, U1 TL074, U2 TL074, U3 TL072

Commit message: chaging 1M to 30k for triangle adjustment
Parts:
- removed G***: LOGO, logos:solisynth_13mm_4000DPI
- D1, D2, D5: value 1N5819HW-7-F -> D
- R29: value 1M -> 30k
